Commit message: [#4]
Nuclear option: changed the overall xacro file.

File: code/simulation/src/uuv_simulator/uuv_sensor_plugins/uuv_sensor_ros_plugins/urdf/pose_3d_snippets.xacro (robot description, xacro)
@@ -32,4 +32,5 @@
     <gazebo>
       <plugin name="pose_3d_plugin" filename="libuuv_gazebo_ros_pose_gt_plugin.so">
+      	<reference_frame>world_ned</reference_frame>
         <robot_namespace>${namespace}</robot_namespace>
         <link_name>${namespace}/base_link</link_name>
