Commit message: [#4]
Updated values of BlueROV2H mass, water density and CoG.

File: code/simulation/src/bluerov2/bluerov2_description/urdf/base.xacro (robot description, xacro)
@@ -13,5 +13,5 @@
   -->
   <!-- Mass -->
-  <xacro:property name="mass" value="11.2"/>
+  <xacro:property name="mass" value="11.26"/>
   <!-- Describing the dimensions of the vehicle's bounding box: width, length, height -->
   <xacro:property name="x_size" value="0.448"/>
@@ -22,5 +22,5 @@
   <xacro:property name="volume" value="0.011054"/>
   <!-- Center of gravity -->
-  <xacro:property name="cog" value="0 0 0"/>
+  <xacro:property name="cog" value="0 0 -0.02"/>
   <!--
   Center of buoyancy according to eq. (3.1) p. 28 in Berg2012.
@@ -28,7 +28,7 @@
   assume NWU (otherwise cob is below cog?). 0.155
   -->
-  <xacro:property name="cob" value="0 0 0.3872"/>
+  <xacro:property name="cob" value="0 0 0.0"/>
   <!-- Fluid density -->
-  <xacro:property name="rho" value="1028"/>
+  <xacro:property name="rho" value="999.97"/>  <!-- Freshwater density, change to 1028.0 if in seawater -->
   <!--
     Visual mesh file for the vehicle, usually in DAE (Collada) format. Be sure to store the

Commit message: [#4]
1) Changed CoB CoG separation.
2) Removed unused parameter in launch file.

File: code/simulation/src/bluerov2/bluerov2_description/urdf/base.xacro (robot description, xacro)
@@ -22,5 +22,5 @@
   <xacro:property name="volume" value="0.011054"/>
   <!-- Center of gravity -->
-  <xacro:property name="cog" value="0 0 -0.02"/>
+  <xacro:property name="cog" value="0 0 0"/>
   <!--
   Center of buoyancy according to eq. (3.1) p. 28 in Berg2012.
@@ -28,5 +28,5 @@
   assume NWU (otherwise cob is below cog?). 0.155
   -->
-  <xacro:property name="cob" value="0 0 0.0"/>
+  <xacro:property name="cob" value="0 0 0.02"/>
   <!-- Fluid density -->
   <xacro:property name="rho" value="999.97"/>  <!-- Freshwater density, change to 1028.0 if in seawater -->

Commit message: [#4]
Modified volume in freshwater.

File: code/simulation/src/bluerov2/bluerov2_description/urdf/base.xacro (robot description, xacro)
@@ -13,5 +13,5 @@
   -->
   <!-- Mass -->
-  <xacro:property name="mass" value="11.26"/>
+  <xacro:property name="mass" value="11.20"/>
   <!-- Describing the dimensions of the vehicle's bounding box: width, length, height -->
   <xacro:property name="x_size" value="0.448"/>
@@ -20,5 +20,5 @@
   <!-- minion_usv_height is not really! It's just for run... We need first calculate the Fossen parameters -->
   <!-- Volume -->
-  <xacro:property name="volume" value="0.011054"/>
+  <xacro:property name="volume" value="0.1127"/> <!-- Neutral in freshwater at 0.11260338, for seawater use 0.011054-->
   <!-- Center of gravity -->
   <xacro:property name="cog" value="0 0 0"/>

Commit message: [#4]
Descresed volume.

File: code/simulation/src/bluerov2/bluerov2_description/urdf/base.xacro (robot description, xacro)
@@ -20,5 +20,5 @@
   <!-- minion_usv_height is not really! It's just for run... We need first calculate the Fossen parameters -->
   <!-- Volume -->
-  <xacro:property name="volume" value="0.1127"/> <!-- Neutral in freshwater at 0.11260338, for seawater use 0.011054-->
+  <xacro:property name="volume" value="0.11261"/> <!-- Neutral in freshwater at 0.11260338, for seawater use 0.011054-->
   <!-- Center of gravity -->
   <xacro:property name="cog" value="0 0 0"/>

Commit message: [#4]
Corrected order of magnitude of the volume.

File: code/simulation/src/bluerov2/bluerov2_description/urdf/base.xacro (robot description, xacro)
@@ -20,5 +20,5 @@
   <!-- minion_usv_height is not really! It's just for run... We need first calculate the Fossen parameters -->
   <!-- Volume -->
-  <xacro:property name="volume" value="0.11261"/> <!-- Neutral in freshwater at 0.11260338, for seawater use 0.011054-->
+  <xacro:property name="volume" value="0.011261"/> <!-- Neutral in freshwater at 0.011260338, for seawater use 0.011054-->
   <!-- Center of gravity -->
   <xacro:property name="cog" value="0 0 0"/>
